File: hardware/Schematic/MSXPi_v0.7.0_Rev_2/msxpi.brd (EAGLE design)
At the start: 101 x 64.7 mm, 21 parts, among them IC1 LD117AS33TR

Commit message: PCB rev 3
Parts:
- added C3: (no value), rcl:E2,5-5
- added CS1, CS12, CS2, GND10, GND11, GND4, GND9, ROMOE1, ROMOE2, ROMOE3: (no value), wirepad:2,15/1,0
Connections:
- new net CS12: CS12.1, JP6.3
- new net CS2: CS2.1, JP6.2
- new net PIN1: EPM3064SLC.1, GND4.1
- new net PIN2: EPM3064SLC.2, GND9.1
- new net PIN43: EPM3064SLC.43, GND10.1
- new net PIN44: EPM3064SLC.44, GND11.1
- new net ROM_OE: 27C256.22, ROMOE1.1, ROMOE2.1, ROMOE3.1
- net CS1: now also CS1.1; no longer 27C256.22
- net GND: now also C3.-
- net VCCIO: now also C3.+
Routing:
- net PIN1: track 0.00 -> 106.7 mm, vias 0 -> 1
- net PIN2: track 0.00 -> 97.3 mm, vias 0 -> 4
- net ROM_OE: track 0.00 -> 71.6 mm
- net CS1: track 80.2 -> 13.2 mm
- net PIN44: track 0.00 -> 52.9 mm, vias 0 -> 5
- net PIN43: track 0.00 -> 29.8 mm, vias 0 -> 1
- net CS12: track 0.00 -> 20.7 mm
- net CS2: track 0.00 -> 16.1 mm
- net D6: track 124.1 -> 117.4 mm
- net GND: track 257.8 -> 251.4 mm
- net A14: track 91.2 -> 85.8 mm
- net +5V: track 202.0 -> 206.4 mm
- net A3: track 85.9 -> 90.0 mm
- net SPI_MOSI_GPIO16: track 45.5 -> 49.1 mm
- net A13: track 89.3 -> 85.8 mm
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Other:
- board text added: "MSX Pi Interface v0.7 Rev.3"
- board text removed: "MSX Pi Interface v0.7 Rev.2"
