File: hardware/Schematic/MSXPi_v0.7.0_Rev_2/msxpi.sch (EAGLE design)
At the start: 21 parts, among them IC1 LD117AS33TR

Commit message: PCB rev 3
Parts:
- added C3: (no value), rcl:CPOL-EUE2.5-5
- added CS1, CS12, CS2, GND10, GND11, GND4, GND9, ROMOE1, ROMOE2, ROMOE3: (no value), wirepad:2,15/1,0
Connections:
- new net CS12: CS12.P, JP6.!CS12
- new net CS2: CS2.P, JP6.!CS2
- new net PIN1: EPM3064SLC.GCLR/, GND4.P
- new net PIN2: EPM3064SLC.OE2-GCLK2, GND9.P
- new net PIN43: EPM3064SLC.GCLK1, GND10.P
- new net PIN44: EPM3064SLC.OE1, GND11.P
- new net ROM_OE: 27C256A.!OE, ROMOE1.P, ROMOE2.P, ROMOE3.P
- net CS1: now also CS1.P; no longer 27C256A.!OE
- net GND: now also C3.-
- net VCCIO: now also C3.+
Changed lines of the file:
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@@
 <part name="+5V" library="wirepad" deviceset="2,15/1,0" device=""/>
 <part name="GND" library="wirepad" deviceset="2,15/1,0" device=""/>
+<part name="ROMOE1" library="wirepad" deviceset="2,15/1,0" device=""/>
+<part name="ROMOE2" library="wirepad" deviceset="2,15/1,0" device=""/>
+<part name="ROMOE3" library="wirepad" deviceset="2,15/1,0" device=""/>
+<part name="CS1" library="wirepad" deviceset="2,15/1,0" device=""/>
+<part name="CS2" library="wirepad" deviceset="2,15/1,0" device=""/>
+<part name="CS12" library="wirepad" deviceset="2,15/1,0" device=""/>
+<part name="GND4" library="wirepad" deviceset="2,15/1,0" device=""/>
+<part name="GND9" library="wirepad" deviceset="2,15/1,0" device=""/>
+<part name="GND10" library="wirepad" deviceset="2,15/1,0" device=""/>
+<part name="GND11" library="wirepad" deviceset="2,15/1,0" device=""/>
+<part name="C3" library="rcl" deviceset="CPOL-EU" device="E2.5-5"/>
 </parts>
 <sheets>
@@
 <attribute name="VALUE" x="158.242" y="-77.343" size="1.778" layer="96" rot="R90"/>
 </instance>
+<instance part="ROMOE1" gate="1" x="-7.62" y="-58.42" smashed="yes" rot="R270">
+<attribute name="VALUE" x="-10.922" y="-57.277" size="1.778" layer="96" rot="R270"/>
+</instance>
+<instance part="ROMOE2" gate="1" x="-2.54" y="-58.42" smashed="yes" rot="R270">
+<attribute name="VALUE" x="-5.842" y="-57.277" size="1.778" layer="96" rot="R270"/>
+</instance>
+<instance part="ROMOE3" gate="1" x="2.54" y="-58.42" smashed="yes" rot="R270">
+<attribute name="VALUE" x="-0.762" y="-57.277" size="1.778" layer="96" rot="R270"/>
+</instance>
+<instance part="CS1" gate="1" x="-7.62" y="-53.34" smashed="yes" rot="R90">
+<attribute name="VALUE" x="-4.318" y="-54.483" size="1.778" layer="96" rot="R90"/>
+</instance>
+<instance part="CS2" gate="1" x="-2.54" y="-53.34" smashed="yes" rot="R90">
+<attribute name="VALUE" x="0.762" y="-54.483" size="1.778" layer="96" rot="R90"/>
+</instance>
+<instance part="CS12" gate="1" x="2.54" y="-53.34" smashed="yes" rot="R90">
+<attribute name="VALUE" x="5.842" y="-54.483" size="1.778" layer="96" rot="R90"/>
+</instance>
+<instance part="GND4" gate="1" x="170.18" y="-76.2" smashed="yes" rot="R90">
+<attribute name="VALUE" x="173.482" y="-77.343" size="1.778" layer="96" rot="R90"/>
+</instance>
+<instance part="GND9" gate="1" x="175.26" y="-76.2" smashed="yes" rot="R90">
+<attribute name="VALUE" x="178.562" y="-77.343" size="1.778" layer="96" rot="R90"/>
+</instance>
+<instance part="GND10" gate="1" x="180.34" y="-76.2" smashed="yes" rot="R90">
+<attribute name="VALUE" x="183.642" y="-77.343" size="1.778" layer="96" rot="R90"/>
+</instance>
+<instance part="GND11" gate="1" x="185.42" y="-76.2" smashed="yes" rot="R90">
+<attribute name="VALUE" x="188.722" y="-77.343" size="1.778" layer="96" rot="R90"/>
+</instance>
+<instance part="C3" gate="G$1" x="83.82" y="-71.12" rot="R180"/>
 </instances>
 <busses>
@@
 <pinref part="C1" gate="G$1" pin="2"/>
 <wire x1="93.98" y1="-68.58" x2="93.98" y2="-63.5" width="0.1524" layer="91"/>
-<wire x1="93.98" y1="-63.5" x2="68.58" y2="-63.5" width="0.1524" layer="91"/>
 <pinref part="IC1" gate="G$1" pin="ADJ"/>
+<wire x1="93.98" y1="-63.5" x2="83.82" y2="-63.5" width="0.1524" layer="91"/>
+<wire x1="83.82" y1="-63.5" x2="68.58" y2="-63.5" width="0.1524" layer="91"/>
 <wire x1="68.58" y1="-63.5" x2="68.58" y2="-68.58" width="0.1524" layer="91"/>
 <wire x1="45.72" y1="-63.5" x2="68.58" y2="-63.5" width="0.1524" layer="91"/>
@@
 <pinref part="GND7" gate="1" pin="GND"/>
 <wire x1="35.56" y1="-63.5" x2="35.56" y2="-81.28" width="0.1524" layer="91"/>
+<pinref part="C3" gate="G$1" pin="-"/>
+<wire x1="83.82" y1="-66.04" x2="83.82" y2="-63.5" width="0.1524" layer="91"/>
+<junction x="83.82" y="-63.5"/>
 </segment>
 <segment>
@@
 <net name="CS1" class="0">
 <segment>
-<pinref part="27C256" gate="A" pin="!OE"/>
-<wire x1="55.88" y1="-15.24" x2="71.12" y2="-15.24" width="0.1524" layer="91"/>
-</segment>
-<segment>
 <pinref part="JP6" gate="CRTRDG" pin="!CS1"/>
 <wire x1="0" y1="-22.86" x2="-5.08" y2="-22.86" width="0.1524" layer="91"/>
 <label x="-10.16" y="-22.86" size="1.778" layer="95"/>
+</segment>
+<segment>
+<pinref part="CS1" gate="1" pin="P"/>
+<wire x1="-7.62" y1="-50.8" x2="-7.62" y2="-45.72" width="0.1524" layer="91"/>
+<label x="-7.62" y="-45.72" size="1.778" layer="95"/>
 </segment>
 </net>
@@
 <segment>
 <pinref part="C1" gate="G$1" pin="1"/>
-<wire x1="83.82" y1="-76.2" x2="93.98" y2="-76.2" width="0.1524" layer="91"/>
 <wire x1="93.98" y1="-76.2" x2="106.68" y2="-76.2" width="0.1524" layer="91"/>
 <junction x="93.98" y="-76.2"/>
@@
 <pinref part="P+2" gate="VCC" pin="VCC"/>
 <label x="106.68" y="-71.12" size="1.778" layer="95"/>
+<pinref part="IC1" gate="G$1" pin="OUT"/>
+<wire x1="76.2" y1="-76.2" x2="83.82" y2="-76.2" width="0.1524" layer="91"/>
+<pinref part="C3" gate="G$1" pin="+"/>
+<wire x1="83.82" y1="-76.2" x2="93.98" y2="-76.2" width="0.1524" layer="91"/>
+<wire x1="83.82" y1="-73.66" x2="83.82" y2="-76.2" width="0.1524" layer="91"/>
+<junction x="83.82" y="-76.2"/>
 </segment>
 <segment>
@@
 <junction x="182.88" y="30.48"/>
 </segment>
-<segment>
-<pinref part="IC1" gate="G$1" pin="OUT"/>
-<wire x1="76.2" y1="-76.2" x2="93.98" y2="-76.2" width="0.1524" layer="91"/>
-</segment>
 </net>
 <net name="TCK" class="0">
@@
 </segment>
 </net>
+<net name="CS2" class="0">
+<segment>
+<pinref part="JP6" gate="CRTRDG" pin="!CS2"/>
+<wire x1="0" y1="-25.4" x2="-5.08" y2="-25.4" width="0.1524" layer="91"/>
+<label x="-10.16" y="-25.4" size="1.778" layer="95"/>
+</segment>
+<segment>
+<pinref part="CS2" gate="1" pin="P"/>
+<wire x1="-2.54" y1="-50.8" x2="-2.54" y2="-45.72" width="0.1524" layer="91"/>
+<label x="-2.54" y="-45.72" size="1.778" layer="95"/>
+</segment>
+</net>
+<net name="CS12" class="0">
+<segment>
+<pinref part="JP6" gate="CRTRDG" pin="!CS12"/>
+<wire x1="0" y1="-27.94" x2="-5.08" y2="-27.94" width="0.1524" layer="91"/>
+<label x="-10.16" y="-27.94" size="1.778" layer="95"/>
+</segment>
+<segment>
+<pinref part="CS12" gate="1" pin="P"/>
+<wire x1="2.54" y1="-50.8" x2="2.54" y2="-45.72" width="0.1524" layer="91"/>
+<label x="2.54" y="-45.72" size="1.778" layer="95"/>
+</segment>
+</net>
+<net name="ROM_OE" class="0">
+<segment>
+<pinref part="27C256" gate="A" pin="!OE"/>
+<wire x1="71.12" y1="-15.24" x2="66.04" y2="-15.24" width="0.1524" layer="91"/>
+<label x="58.42" y="-15.24" size="1.778" layer="95"/>
+</segment>
+<segment>
+<pinref part="ROMOE1" gate="1" pin="P"/>
+<wire x1="-7.62" y1="-60.96" x2="-7.62" y2="-63.5" width="0.1524" layer="91"/>
+<wire x1="-7.62" y1="-63.5" x2="-2.54" y2="-63.5" width="0.1524" layer="91"/>
+<pinref part="ROMOE2" gate="1" pin="P"/>
+<wire x1="-2.54" y1="-63.5" x2="-2.54" y2="-60.96" width="0.1524" layer="91"/>
+<pinref part="ROMOE3" gate="1" pin="P"/>
+<wire x1="2.54" y1="-60.96" x2="2.54" y2="-63.5" width="0.1524" layer="91"/>
+<wire x1="2.54" y1="-63.5" x2="-2.54" y2="-63.5" width="0.1524" layer="91"/>
+<junction x="-2.54" y="-63.5"/>
+<label x="2.54" y="-66.04" size="1.778" layer="95"/>
+</segment>
+</net>
+<net name="PIN43" class="0">
+<segment>
+<pinref part="EPM3064SLC" gate="0" pin="GCLK1"/>
+<wire x1="152.4" y1="48.26" x2="147.32" y2="48.26" width="0.1524" layer="91"/>
+<label x="142.24" y="48.26" size="1.778" layer="95"/>
+</segment>
+<segment>
+<pinref part="GND10" gate="1" pin="P"/>
+<wire x1="180.34" y1="-73.66" x2="180.34" y2="-68.58" width="0.1524" layer="91"/>
+<label x="177.8" y="-68.58" size="1.778" layer="95"/>
+</segment>
+</net>
+<net name="PIN1" class="0">
+<segment>
+<pinref part="EPM3064SLC" gate="0" pin="GCLR/"/>
+<wire x1="152.4" y1="45.72" x2="147.32" y2="45.72" width="0.1524" layer="91"/>
+<label x="142.24" y="45.72" size="1.778" layer="95"/>
+</segment>
+<segment>
+<pinref part="GND4" gate="1" pin="P"/>
+<wire x1="170.18" y1="-73.66" x2="170.18" y2="-68.58" width="0.1524" layer="91"/>
+<label x="167.64" y="-68.58" size="1.778" layer="95"/>
+</segment>
+</net>
+<net name="PIN44" class="0">
+<segment>
+<pinref part="EPM3064SLC" gate="0" pin="OE1"/>
+<wire x1="152.4" y1="43.18" x2="147.32" y2="43.18" width="0.1524" layer="91"/>
+<label x="142.24" y="43.18" size="1.778" layer="95"/>
+</segment>
+<segment>
+<pinref part="GND11" gate="1" pin="P"/>
+<wire x1="185.42" y1="-73.66" x2="185.42" y2="-68.58" width="0.1524" layer="91"/>
+<label x="182.88" y="-68.58" size="1.778" layer="95"/>
+</segment>
+</net>
+<net name="PIN2" class="0">
+<segment>
+<pinref part="EPM3064SLC" gate="0" pin="OE2-GCLK2"/>
+<wire x1="152.4" y1="40.64" x2="147.32" y2="40.64" width="0.1524" layer="91"/>
+<label x="142.24" y="40.64" size="1.778" layer="95"/>
+</segment>
+<segment>
+<pinref part="GND9" gate="1" pin="P"/>
+<wire x1="175.26" y1="-73.66" x2="175.26" y2="-68.58" width="0.1524" layer="91"/>
+<label x="172.72" y="-68.58" size="1.778" layer="95"/>
+</segment>
+</net>
