File: hardware/Schematic/MSXPi_v0.7.0_Rev_4/msxpi.brd (EAGLE design)
At the start: 101 x 64.7 mm, 21 parts, among them IC1 LD117AS33TR

Commit message: v20170705.00060 with MSXPi-DOS, NFS, TOOLS and schematic v0.7 Rev.4
Parts:
- added A14, A15, CS1, CS12, CS2, GND10, GND11, GND4, GND9, ROMOE1, ROMOE2, ROMOE3, ROM_OE: (no value), wirepad:2,15/1,0
- added C3: (no value), rcl:E2,5-5
Connections:
- new net A15: A15.1, JP6.18
- new net CS12: CS12.1, JP6.3
- new net CS2: CS2.1, JP6.2
- new net PIN1: EPM3064SLC.1, GND4.1
- new net PIN2: EPM3064SLC.2, GND9.1
- new net PIN43: EPM3064SLC.43, GND10.1
- new net PIN44: EPM3064SLC.44, GND11.1
- new net ROM_A14: 27C256.27, ROM_OE.1
- new net ROM_OE: 27C256.22, ROMOE1.1, ROMOE2.1, ROMOE3.1
- net A14: now also A14.1; no longer 27C256.27
- net CS1: now also CS1.1; no longer 27C256.22
- net GND: now also C3.-
- net VCCIO: now also C3.+
Routing:
- net PIN1: track 0.00 -> 106.7 mm, vias 0 -> 1
- net PIN2: track 0.00 -> 97.3 mm, vias 0 -> 4
- net ROM_OE: track 0.00 -> 71.6 mm
- net CS1: track 80.2 -> 13.2 mm
- net PIN44: track 0.00 -> 52.9 mm, vias 0 -> 5
- net A15: track 0.00 -> 44.4 mm, vias 0 -> 2
- net ROM_A14: track 0.00 -> 41.4 mm, vias 0 -> 1
- net PIN43: track 0.00 -> 29.8 mm, vias 0 -> 1
- net A14: track 91.2 -> 69.4 mm, vias 2 -> 3
- net CS12: track 0.00 -> 20.7 mm
- net CS2: track 0.00 -> 16.1 mm
- net GND: track 257.8 -> 250.7 mm
- net D6: track 124.1 -> 117.4 mm
- net +5V: track 202.0 -> 206.4 mm
- net A3: track 85.9 -> 90.0 mm
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Other:
- board text added: "MSX Pi Interface v0.7 Rev.4"
- board text added: "MSXPi"
- board text added: "v0.7 Rev.4"
- board text removed: "MSX Pi Interface v0.7 Rev.2"
