File: hardware/Schematic/MSXPi_v0.7.0_Rev_4/msxpi.brd (EAGLE design)
At the start: 101 x 64.7 mm, 32 parts, among them IC1 LD117AS33TR

Commit message: master branch now contain latest develoment branch, v20170705.00060. Contain MSXP-DOS, Tools, NFS, disk images
Parts:
- added A14, A15, ROM_OE: (no value), wirepad:2,15/1,0
Connections:
- new net A15: A15.1, JP6.18
- new net ROM_A14: 27C256.27, ROM_OE.1
- net A14: now also A14.1; no longer 27C256.27
Routing:
- net A15: track 0.00 -> 44.4 mm, vias 0 -> 2
- net ROM_A14: track 0.00 -> 41.4 mm, vias 0 -> 1
- net A14: track 85.8 -> 69.4 mm, vias 2 -> 3
- net GND: track 251.4 -> 250.7 mm
Other:
- board text added: "MSX Pi Interface v0.7 Rev.4"
- board text added: "MSXPi"
- board text added: "v0.7 Rev.4"
- board text removed: "MSX Pi Interface v0.7 Rev.3"
