File: hardware/Schematic/MSXPi_v0.7.0_Rev_4/msxpi.sch (EAGLE design)
At the start: 21 parts, among them IC1 LD117AS33TR

Commit message: v20170705.00060 with MSXPi-DOS, NFS, TOOLS and schematic v0.7 Rev.4
Parts:
- added A14, A15, CS1, CS12, CS2, GND10, GND11, GND4, GND9, ROMOE1, ROMOE2, ROMOE3, ROM_OE: (no value), wirepad:2,15/1,0
- added C3: (no value), rcl:CPOL-EUE2.5-5
- R1: device rcl:R-EU_0207/7 -> rcl:R-US_0207/7
Connections:
- new net A15: A15.P, JP6.A15
- new net CS12: CS12.P, JP6.!CS12
- new net CS2: CS2.P, JP6.!CS2
- new net PIN1: EPM3064SLC.GCLR/, GND4.P
- new net PIN2: EPM3064SLC.OE2-GCLK2, GND9.P
- new net PIN43: EPM3064SLC.GCLK1, GND10.P
- new net PIN44: EPM3064SLC.OE1, GND11.P
- new net ROM_A14: 27C256A.A14, ROM_OE.P
- new net ROM_OE: 27C256A.!OE, ROMOE1.P, ROMOE2.P, ROMOE3.P
- net A14: now also A14.P; no longer 27C256A.A14
- net CS1: now also CS1.P; no longer 27C256A.!OE
- net GND: now also C3.-
- net VCCIO: now also C3.+
