File: hardware/Schematic/MSXPi_v0.7.0_Rev_6/msxpi.brd (EAGLE design)
At the start: 101 x 64.7 mm, 37 parts, among them IC1 LD117AS33TR

Commit message: Schematic Revision 6
Parts:
- added R6: (no value), rcl:0207/7
- moved C4 6.67 mm to (94.8, 63.8)
Connections:
- net +5V: now also R6.2
- net ROM_OE: now also R6.1
Routing:
- net GND: track 268.5 -> 263.4 mm, vias 7 -> 6
- net +5V: track 226.1 -> 229.7 mm, vias 2 -> 3
- net ROM_OE: track 67.4 -> 71.1 mm
Other:
- board text added: "MSX Pi Interface v0.7 Rev.6"
- board text added: "v0.7 Rev.6"
- board text removed: "MSX Pi Interface v0.7 Rev.5"
- board text removed: "v0.7 Rev.5"
Changed lines of the file:
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@@
 <board>
 <plain>
-<text x="62.23" y="69.85" size="1.016" layer="16" font="vector" rot="MR0">MSX Pi Interface v0.7 Rev.5</text>
+<text x="62.23" y="69.85" size="1.016" layer="16" font="vector" rot="MR0">MSX Pi Interface v0.7 Rev.6</text>
 <text x="15.367" y="19.558" size="0.8128" layer="1" font="vector">Ronivon Costa, 2017
 http://Retro-CPU.run</text>
@@
 <rectangle x1="0.0239875" y1="0.035653125" x2="0.02530625" y2="0.03584375" layer="200"/>
 <rectangle x1="-0.00009375" y1="0.035653125" x2="0.0239875" y2="0.03584375" layer="201"/>
-<text x="72.635825" y="28.650921875" size="1.524" layer="1" font="vector" ratio="9" distance="43">v0.7 Rev.5</text>
+<text x="72.635825" y="28.650921875" size="1.524" layer="1" font="vector" ratio="9" distance="43">v0.7 Rev.6</text>
 </plain>
 <attributes>
@@
 <element name="A14" library="wirepad" package="2,15/1,0" value="" x="95.25" y="34.29"/>
 <element name="R1" library="rcl" package="0207/7" value="" x="27.94" y="69.85"/>
-<element name="C4" library="capacitor-wima" package="C2.5-3" value="" x="101.061603125" y="65.928" rot="R270"/>
+<element name="C4" library="capacitor-wima" package="C2.5-3" value="" x="94.757671875" y="63.7631" rot="R270"/>
 <element name="JP1" library="jumper" package="JP1" value="" x="88.663134375" y="40.823084375" rot="R90"/>
 <element name="JP2" library="jumper" package="JP1" value="" x="20.723003125" y="63.875790625" smashed="yes" rot="R180">
@@
 <attribute name="VALUE" x="17.802003125" y="66.415790625" size="1.27" layer="27" ratio="10" rot="R270"/>
 </element>
+<element name="R6" library="rcl" package="0207/7" value="" x="77.82000625" y="65.31391875" rot="R180"/>
 </elements>
 <signals>
@@
 <wire x1="92.964" y1="68.326" x2="92.964" y2="67.564" width="0.1524" layer="16"/>
 <wire x1="92.964" y1="67.564" x2="91.44" y2="66.04" width="0.1524" layer="16"/>
-<wire x1="91.44" y1="66.04" x2="73.66" y2="66.04" width="0.1524" layer="16"/>
-<wire x1="73.66" y1="66.04" x2="67.31" y2="59.69" width="0.1524" layer="16"/>
-<wire x1="67.31" y1="59.69" x2="64.77" y2="59.69" width="0.1524" layer="16"/>
-<wire x1="64.77" y1="59.69" x2="62.23" y2="57.15" width="0.1524" layer="16"/>
-<wire x1="62.23" y1="57.15" x2="62.23" y2="49.276" width="0.1524" layer="16"/>
+<wire x1="62.23" y1="57.439259375" x2="62.23" y2="49.276" width="0.1524" layer="16"/>
 <wire x1="62.23" y1="49.276" x2="61.976" y2="49.022" width="0.1524" layer="16"/>
+<wire x1="91.44" y1="66.04" x2="91.44" y2="66.03349375" width="0.1524" layer="16"/>
+<wire x1="91.44" y1="66.03349375" x2="89.598746875" y2="64.192240625" width="0.1524" layer="16"/>
+<wire x1="89.598746875" y1="64.192240625" x2="84.70208125" y2="64.192240625" width="0.1524" layer="16"/>
+<wire x1="62.23" y1="57.439259375" x2="64.448296875" y2="59.65755625" width="0.1524" layer="16"/>
+<wire x1="64.448296875" y1="59.65755625" x2="80.167396875" y2="59.65755625" width="0.1524" layer="16"/>
+<wire x1="80.167396875" y1="59.65755625" x2="84.70208125" y2="64.192240625" width="0.1524" layer="16"/>
 </signal>
 <signal name="A2">
@@
 <contactref element="C4" pad="2"/>
 <wire x1="94.066453125" y1="55.539546875" x2="94.107" y2="55.499" width="0.1524" layer="1"/>
-<wire x1="101.061603125" y1="64.658" x2="100.55845625" y2="64.658" width="0.1524" layer="1"/>
-<wire x1="100.55845625" y1="64.658" x2="97.608525" y2="61.70806875" width="0.1524" layer="1"/>
-<via x="97.608525" y="61.70806875" extent="1-16" drill="0.6096" shape="octagon"/>
-<wire x1="97.608525" y1="61.70806875" x2="97.550390625" y2="61.70806875" width="0.1524" layer="16"/>
-<wire x1="97.550390625" y1="61.70806875" x2="94.1054" y2="58.263078125" width="0.1524" layer="16"/>
-<wire x1="94.1054" y1="58.263078125" x2="94.1054" y2="55.5006" width="0.1524" layer="16"/>
-<wire x1="94.1054" y1="55.5006" x2="94.107" y2="55.499" width="0.1524" layer="16"/>
 <wire x1="39.0906" y1="13.335" x2="38.66269375" y2="13.335" width="0.254" layer="16"/>
 <wire x1="38.66269375" y1="13.335" x2="38.66269375" y2="19.156003125" width="0.254" layer="16"/>
 <wire x1="38.66269375" y1="19.156003125" x2="36.83" y2="19.156003125" width="0.254" layer="16"/>
 <wire x1="94.107" y1="48.387" x2="92.71" y2="46.99" width="0.254" layer="1"/>
+<wire x1="94.1054" y1="55.5006" x2="94.107" y2="55.499" width="0.1524" layer="16"/>
+<wire x1="94.757671875" y1="62.4931" x2="94.757671875" y2="58.257809375" width="0.1524" layer="1"/>
+<wire x1="94.757671875" y1="58.257809375" x2="94.187428125" y2="57.687565625" width="0.1524" layer="1"/>
+<wire x1="94.187428125" y1="57.687565625" x2="94.187428125" y2="55.579428125" width="0.1524" layer="1"/>
+<wire x1="94.187428125" y1="55.579428125" x2="94.107" y2="55.499" width="0.1524" layer="1"/>
 </signal>
 <signal name="A6">
@@
 <wire x1="94.869" y1="71.501" x2="97.79" y2="68.58" width="0.1524" layer="1"/>
 <contactref element="C4" pad="1"/>
-<wire x1="101.061603125" y1="67.198" x2="100.05130625" y2="68.52468125" width="0.254" layer="1"/>
-<wire x1="100.05130625" y1="68.52468125" x2="99.257740625" y2="68.628340625" width="0.254" layer="1"/>
-<wire x1="99.257740625" y1="68.628340625" x2="97.761103125" y2="68.663796875" width="0.254" layer="1"/>
-<wire x1="97.761103125" y1="68.663796875" x2="97.79" y2="68.58" width="0.254" layer="1"/>
-<wire x1="97.79" y1="68.58" x2="97.79" y2="63.46388125" width="0.1524" layer="1"/>
-<wire x1="97.79" y1="63.46388125" x2="96.784575" y2="62.45845625" width="0.1524" layer="1"/>
-<wire x1="96.784575" y1="62.45845625" x2="96.461071875" y2="62.134953125" width="0.1524" layer="1"/>
 <wire x1="34.0106" y1="13.335" x2="33.91296875" y2="13.335" width="0.254" layer="16"/>
 <wire x1="33.91296875" y1="13.335" x2="33.91296875" y2="19.156003125" width="0.254" layer="16"/>
@@
 <contactref element="JP1" pad="1"/>
 <wire x1="95.98470625" y1="45.415525" x2="95.98470625" y2="45.41439375" width="0.1524" layer="1"/>
-<wire x1="64.897" y1="71.501" x2="94.869" y2="71.501" width="0.1524" layer="1"/>
+<wire x1="64.897" y1="71.501" x2="73.765821875" y2="71.501" width="0.1524" layer="1"/>
+<wire x1="74.06195" y1="71.501" x2="94.869" y2="71.501" width="0.1524" layer="1"/>
 <wire x1="95.98470625" y1="45.41439375" x2="91.28653125" y2="40.71621875" width="0.1524" layer="1"/>
 <wire x1="91.28653125" y1="40.71621875" x2="90.04" y2="40.71621875" width="0.1524" layer="1"/>
 <wire x1="90.04" y1="40.71621875" x2="89.933134375" y2="40.823084375" width="0.1524" layer="1"/>
-<wire x1="95.98470625" y1="45.415525" x2="96.412159375" y2="45.415525" width="0.1524" layer="1"/>
-<wire x1="96.412159375" y1="45.415525" x2="96.9410125" y2="45.944378125" width="0.1524" layer="1"/>
-<wire x1="96.9410125" y1="45.944378125" x2="96.9410125" y2="48.260165625" width="0.1524" layer="1"/>
-<wire x1="96.9410125" y1="48.260165625" x2="96.374528125" y2="48.82665" width="0.1524" layer="1"/>
-<wire x1="96.374528125" y1="48.82665" x2="96.374528125" y2="62.048409375" width="0.1524" layer="1"/>
-<wire x1="96.374528125" y1="62.048409375" x2="96.461071875" y2="62.134953125" width="0.1524" layer="1"/>
+<wire x1="97.79" y1="68.58" x2="97.79" y2="68.065428125" width="0.1524" layer="1"/>
+<wire x1="97.79" y1="68.065428125" x2="94.757671875" y2="65.0331" width="0.1524" layer="1"/>
+<wire x1="96.63378125" y1="63.156990625" x2="96.63378125" y2="50.745471875" width="0.1524" layer="1"/>
+<wire x1="95.98470625" y1="45.415525" x2="96.3617375" y2="45.415525" width="0.1524" layer="1"/>
+<wire x1="96.3617375" y1="45.415525" x2="96.95041875" y2="46.00420625" width="0.1524" layer="1"/>
+<wire x1="96.95041875" y1="46.00420625" x2="96.95041875" y2="50.428834375" width="0.1524" layer="1"/>
+<wire x1="96.95041875" y1="50.428834375" x2="96.63378125" y2="50.745471875" width="0.1524" layer="1"/>
+<wire x1="96.63378125" y1="63.156990625" x2="94.757671875" y2="65.0331" width="0.1524" layer="1"/>
+<contactref element="R6" pad="2"/>
+<wire x1="74.01000625" y1="65.31391875" x2="74.01000625" y2="66.43185" width="0.1524" layer="16"/>
+<wire x1="74.01000625" y1="66.43185" x2="73.62904375" y2="66.8128125" width="0.1524" layer="16"/>
+<wire x1="73.62904375" y1="66.8128125" x2="73.62904375" y2="71.364221875" width="0.1524" layer="16"/>
+<wire x1="73.62904375" y1="71.364221875" x2="73.765821875" y2="71.501" width="0.1524" layer="16"/>
+<via x="73.765821875" y="71.501" extent="1-16" drill="0.762"/>
+<wire x1="73.765821875" y1="71.501" x2="74.06195" y2="71.501" width="0.1524" layer="1"/>
 </signal>
 <signal name="VCCIO">
@@
 <wire x1="99.83061875" y1="44.341446875" x2="99.83061875" y2="48.26734375" width="0.1524" layer="16"/>
 <wire x1="99.83061875" y1="48.26734375" x2="99.822" y2="48.2759625" width="0.1524" layer="16"/>
+<contactref element="R6" pad="1"/>
+<wire x1="82.55" y1="68.58" x2="82.55" y2="66.2339125" width="0.1524" layer="16"/>
+<wire x1="82.55" y1="66.2339125" x2="81.63000625" y2="65.31391875" width="0.1524" layer="16"/>
 </signal>
 <signal name="PIN43">
