File: hardware/Schematic/MSXPi_v1.0_Rev1/MSXPi1.kicad_pcb (KiCad board)
At the start: 2 copper layers, 102.6 x 65.3 mm, 32 parts, among them J1 Raspberry_Pi_Zero_2_3, J2 JTAG, J3 Conn_02x07_Odd_Even, P1 MSX_CONNECTOR, U1 EPM3064ALC44-10

Commit message: PCB small change
Parts:
- R5: value R_US -> 270R
- renumbered LD1117 to LD1117S33, AT28C256 to U2
Connections:
- J3 pad 1: A14 -> SLTSL
- J3 pad 10: ROM_OE -> mem_oe
- J3 pad 11: wr -> A14
- J3 pad 12: mem_we -> ROM_A14
- J3 pad 13: sltsl -> A15
- J3 pad 14: mem_ce -> ROM_A14
- J3 pad 2: ROM_A14 -> mem_ce
- J3 pad 3: A15 -> WR
- J3 pad 4: ROM_A14 -> mem_we
- J3 pad 6: ROM_OE -> mem_oe
- J3 pad 8: ROM_OE -> mem_oe
Routing:
- net SLTSL: track 0.00 -> 30.0 mm, vias 0 -> 2
- net WR: track 54.8 -> 80.1 mm, vias 0 -> 1
- net mem_oe: track 12.3 -> 28.6 mm, vias 0 -> 1
- net mem_we: track 41.1 -> 26.3 mm
- net ROM_A14: track 24.6 -> 38.4 mm
- net A14: track 56.2 -> 67.6 mm
- net A15: track 36.4 -> 28.0 mm, vias 1 -> 0
- net mem_ce: track 45.0 -> 36.8 mm
- net ROM_OE: track 5.08 -> 0.00 mm
- net CS12: track 16.0 -> 18.2 mm, vias 0 -> 1
- net A6: track 109.0 -> 107.4 mm
- net A13: track 55.2 -> 56.2 mm
- net WAIT: track 77.7 -> 78.5 mm
- net A9: track 41.1 -> 40.4 mm
- net RD: track 52.7 -> 53.3 mm
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