File: hardware/Schematic/MSXPi_v1.0_Rev2/MSXPi1.kicad_pcb (KiCad board)
At the start: 2 copper layers, 102.6 x 65.3 mm, 32 parts, among them J1 Raspberry_Pi_Zero_2_3, J2 JTAG, J3 Conn_02x07_Odd_Even, P1 MSX_CONNECTOR, U1 EPM3064ALC44-10, U2 AT28C256-15PU

Commit message: Schematic and PCB Rev2. Added 2 more LEDs connected to RPi GPIO
Parts:
- added D2: LED, LED_THT:LED_D3.0mm, F.Cu at (118.6, 71.9)
- added D3: LED, LED_THT:LED_D3.0mm, F.Cu at (123.2, 71.9)
- added R14: 270R, Resistor_THT:R_Axial_DIN0204_L3.6mm_D1.6mm_P5.08mm_Horizontal, F.Cu at (131.3, 74.2)
- added R15: 270R, Resistor_THT:R_Axial_DIN0204_L3.6mm_D1.6mm_P5.08mm_Horizontal, F.Cu at (133.6, 74.2)
- moved R5 12.7 mm to (135.9, 74.2), turned to 90 degrees
- moved D1 9.49 mm to (127.8, 71.9), turned to 90 degrees
Connections:
- J1 pad 35: Net-(J1-Pad35) -> RPI_BUSY
- J1 pad 37: Net-(J1-Pad37) -> RPI_ON
Routing:
- net Net-(D2-Pad2): track 0.00 -> 15.0 mm
- net RPI_ON: track 0.00 -> 13.0 mm, vias 0 -> 1
- net Net-(D3-Pad2): track 0.00 -> 13.0 mm
- net RPI_BUSY: track 0.00 -> 12.3 mm
- net GNDREF: track 414.0 -> 423.5 mm
- net Net-(D1-Pad2): track 2.80 -> 10.1 mm
- net SPI_CS: track 77.3 -> 70.5 mm
Other:
- board text added: "MSXPi v1.0 Rev.2 Ronivon Costa, August 2020."
- board text removed: "MSXPi v1.0 Rev.1 Ronivon Costa, August 2020."
