File: hardware/Schematic/MSXPi_v1.1_Rev_1/MSXPi1.sch (KiCad schematic (older format))
At the start: 46 parts, among them J1 Raspberry_Pi_Zero_2_3, J2 JTAG, J3 Conn_02x07_Odd_Even, J4 Conn_02x06_Odd_Even, J5 SJ-2509N, P1 MSX_CONNECTOR, U1 EPM3064ALC44-10, U2 AT28C256-15PU

Commit message: Changed CPLD foot print
Parts:
- U1: footprint MyFootprints:PLCC-44_16.6x16.6mm_P1.27mm -> MyFootprints:PLCC127P1765X1765X457-44N
Other:
- note added: "1"
- note removed: "0"
Changed lines of the file:
@@
 July, 2020
 Text Notes 10650 7650 0    59   ~ 12
-0
+1
 Text Notes 7100 6700 0    59   ~ 12
 Ronivon Costa
@@
 F 0 "U1" H 5450 4515 50  0000 C CNN
 F 1 "EPM3064ALC44-10" H 5450 4424 50  0000 C CNN
-F 2 "MyFootprints:PLCC-44_16.6x16.6mm_P1.27mm" H 5450 2750 50  0001 L BNN
+F 2 "MyFootprints:PLCC127P1765X1765X457-44N" H 5450 2750 50  0001 L BNN
 F 3 "Altera" H 5450 2750 50  0001 L BNN
 F 4 "1549412" H 5450 2750 50  0001 L BNN "Field4"
