File: hardware/Schematic/MSXPi1.kicad_pcb (KiCad board)
At the start: 2 copper layers, 102.6 x 65.3 mm, 48 parts, among them J1 Raspberry_Pi_Zero_2_3, J2 JTAG, J3 Conn_02x07_Odd_Even, J4 Conn_02x06_Odd_Even, J5 SJ-2509N, P1 MSX_CONNECTOR, U1 EPM3064ALC44-10, U2 AT28C256-15PU

Commit message: PCB v1.1 Rev2
Parts:
- moved R15 9.37 mm to (110.0, 73.9)
- moved D2 7.27 mm to (113.8, 70.4), turned to 180 degrees
- moved R14 6.83 mm to (123.7, 69.1), turned to 270 degrees
- moved D1 3.41 mm to (118.9, 70.4), turned to 180 degrees
- moved D3 2.96 mm to (108.7, 70.4), turned to 180 degrees
- moved R5 2.34 mm to (121.4, 69.1), turned to 270 degrees
- renumbered U2 to AT28C256
Routing:
- net RPI_BUSY: track 8.72 -> 18.7 mm
- net GNDREF: track 500.7 -> 492.9 mm
- net Net-(D3-Pad2): track 10.4 -> 6.03 mm
- net Net-(D1-Pad2): track 3.77 -> 5.67 mm
- net SPI_CS: track 37.7 -> 39.3 mm
- net RPI_ON: track 8.18 -> 9.23 mm
Other:
- board text added: "MSXPi v1.1 Rev.2 Ronivon Costa, September 2020."
- board text removed: "MSXPi v1.1 Rev.1 Ronivon Costa, September 2020."

Commit message: Added github url to pcb
Other:
- board text added: "https://github.com/costarc/MSXPi"
Changed lines of the file:
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@@
   (general
     (thickness 1.6)
-    (drawings 29)
+    (drawings 30)
     (tracks 1471)
     (zones 0)
@@
   )
   (setup
-    (last_trace_width 0.5)
+    (last_trace_width 0.25)
     (user_trace_width 0.3)
     (user_trace_width 0.35)
@@
     )
   )
+  (gr_text https://github.com/costarc/MSXPi (at 148.844 83.566) (layer B.SilkS)
+    (effects (font (size 1.5 1.5) (thickness 0.3)) (justify mirror))
+  )
   (gr_text MSXPi (at 151.384 117.348) (layer F.SilkS)
