File: hardware/Schematic/MSXPi_v1.0.1_Rev.0/msxpi.kicad_sch (KiCad schematic)
At the start: 37 parts, among them IC1 LD117A, J1 ROM_SWITCH, U1 AT28C256

Commit message: Cartridge schematic in Kicad 6 and routed. EEPROM is now AT28C256
Parts:
- removed GMOUNT1, GND3, GND4, MOUNT1: 2,15/1,0, msxpi:2,15_1,0, symbol msxpi-eagle-import:2,15/1,0
- added MOUNTHOLE3, MOUNTHOLE4, MOUNTHOLE5: 2,15/1,0, msxpi:2,15_1,0, symbol msxpi-eagle-import:2,15/1,0
- JP2: footprint Connector_PinHeader_2.54mm:PinHeader_2x05_P2.54mm_Vertical -> Connector_IDC:IDC-Header_2x05_P2.54mm_Horizontal
- renumbered GND1 to MOUNTHOLE1, GND2 to MOUNTHOLE2
Connections:
- net SW2 is gone; now on an unnamed net: JP1.46 (SW@2)
- net D3: now also EPM3064ALC44.39 (IO57)
- net D5: now also EPM3064ALC44.41 (IO64)
- net SPI_RDY: now also EPM3064ALC44.40 (IO62)
- net +12V: no longer names the net of JP1.48 (+12V)
- net -12V: no longer names the net of JP1.50 (-12V)
- net GCLR: no longer names the net of MOUNTHOLE1.1 (P)
- net OE2: no longer names the net of MOUNTHOLE2.1 (P)
- net SOUNDIN: no longer names the net of JP1.49 (SOUNDIN)
- net SW1: no longer names the net of JP1.44 (SW@1)
- no-connect marks 2 -> 15
Other:
- note added: "MSXPi Interface V1.0.1 Rev.0 RCC @ 2022 MSXPi interface - connect MSX computer to Raspberry Pi EEPROM AT28C256 re-writeatable from MSX-DOS EEPROM software: https://github.com/costarc/msxcart_flash32k"
- note added: "Mounting holes for RPI"
- note removed: "2 x mount holes to provide support for top side of the Raspberry Pi"
- note removed: "These 4 pads are for experimentation with the corresponding CPLD signals These are not used by the MSXPi"
- company: (none) -> RCC
- title: (none) -> MSXPi
- moved on the sheet: C1, C2, C3, C4, C5, C6, C7, C8, C9, EPM3064ALC44, IC1, J1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
