File: hardware/Schematic/MSXPi_v1.0.1/msxpi.kicad_sch (KiCad schematic)
At the start: 36 parts, among them IC1 LD117A, J1 ROM_SWITCH, U1 AT28C256

Commit message: v1.0.1 Rev 1 - Added some silk that was missing
Other:
- note added: "MSXPi Interface V1.0.1 Rev.1 RCC @ 2022 MSXPi interface - connect MSX computer to Raspberry Pi EEPROM AT28C256 re-writeatable from MSX-DOS EEPROM software: https://github.com/costarc/msxcart_flash32k"
- note removed: "MSXPi Interface V1.0.1 Rev.0 RCC @ 2022 MSXPi interface - connect MSX computer to Raspberry Pi EEPROM AT28C256 re-writeatable from MSX-DOS EEPROM software: https://github.com/costarc/msxcart_flash32k"
Changed lines of the file:
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@@
     (effects (font (size 1 1)) (justify left bottom))
   )
-  (text "MSXPi Interface V1.0.1 Rev.0\nRCC @ 2022\n\nMSXPi interface - connect MSX computer to Raspberry Pi\nEEPROM AT28C256 re-writeatable from MSX-DOS\nEEPROM software: https://github.com/costarc/msxcart_flash32k\n\n"
+  (text "MSXPi Interface V1.0.1 Rev.1\nRCC @ 2022\n\nMSXPi interface - connect MSX computer to Raspberry Pi\nEEPROM AT28C256 re-writeatable from MSX-DOS\nEEPROM software: https://github.com/costarc/msxcart_flash32k\n\n"
     (at 210.058 197.612 0)
     (effects (font (size 1.27 1.27)) (justify left bottom))

Commit message: Updated dates in schematics
Other:
- note added: "MSXPi Interface V1.0.1 Rev.1 RCC @ 2022 MSXPi interface - connect MSX computer to Raspberry Pi EEPROM AT28C256 re-writeatable from MSX-DOS EEPROM software: https://github.com/costarc/msxcart_flash32k 2022-12-25"
- note removed: "MSXPi Interface V1.0.1 Rev.1 RCC @ 2022 MSXPi interface - connect MSX computer to Raspberry Pi EEPROM AT28C256 re-writeatable from MSX-DOS EEPROM software: https://github.com/costarc/msxcart_flash32k"
Changed lines of the file:
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@@
     (effects (font (size 1 1)) (justify left bottom))
   )
-  (text "MSXPi Interface V1.0.1 Rev.1\nRCC @ 2022\n\nMSXPi interface - connect MSX computer to Raspberry Pi\nEEPROM AT28C256 re-writeatable from MSX-DOS\nEEPROM software: https://github.com/costarc/msxcart_flash32k\n\n"
+  (text "MSXPi Interface V1.0.1 Rev.1\nRCC @ 2022\n\nMSXPi interface - connect MSX computer to Raspberry Pi\nEEPROM AT28C256 re-writeatable from MSX-DOS\nEEPROM software: https://github.com/costarc/msxcart_flash32k\n\n2022-12-25"
     (at 210.058 197.612 0)
     (effects (font (size 1.27 1.27)) (justify left bottom))

Commit message: Minimnized jumpers - SLTSL and A14/A15 only
Parts:
- removed R6: 10k, msxpi:0207_7, symbol msxpi-eagle-import:R-US_0207/7
- added J2: WRITE_EN, Connector_PinHeader_2.54mm:PinHeader_1x02_P2.54mm_Vertical, symbol Connector_Generic:Conn_02x01
- J1: footprint Connector_PinHeader_2.54mm:PinHeader_2x07_P2.54mm_Vertical -> Connector_PinHeader_2.54mm:PinHeader_2x03_P2.54mm_Vertical; symbol Connector_Generic:Conn_02x07_Odd_Even -> Connector_Generic:Conn_02x03_Odd_Even
- JP1: footprint Roni Footprints:MSX_CART -> Roni Footprints:MSX_CART_SW
Connections:
- net /CS1: no longer J1.13 (Pin_13)
- net /CS12: no longer J1.9 (Pin_9)
- net /CS2: no longer J1.11 (Pin_11)
- net /MEM_CE: now also J1.2 (Pin_2); no longer J1.8 (Pin_8)
- net /MEM_WE: now also J2.2 (Pin_2); no longer J1.2 (Pin_2)
- net /RD: now also U1.22 (~{OE})
- net /SLTSL: now also J1.1 (Pin_1); no longer J1.7 (Pin_7)
- net /WR: now also J2.1 (Pin_1); no longer J1.1 (Pin_1)
- removed net /MEM_OE: J1.10 (Pin_10), J1.12 (Pin_12), J1.14 (Pin_14), U1.22 (~{OE})
Other:
- note added: "Jumpers to select ROM Bank, and enable the EEPROM for writing. J2 is optional (may be permanently closed with solder) since write protection is controlled via software."
- note added: "MSXPi Interface V1.0.1 Rev.2 RCC @ 2017 - 2023 MSXPi interface - connect MSX computer to Raspberry Pi EEPROM AT28C256 re-writeatable from MSX-DOS EEPROM software: https://github.com/costarc/msxcart_flash32k 2023-02-26"
- note removed: "Jumpers to select ROM Bank, and enable the EEPROM for writing."
- note removed: "MSXPi Interface V1.0.1 Rev.1 RCC @ 2022 MSXPi interface - connect MSX computer to Raspberry Pi EEPROM AT28C256 re-writeatable from MSX-DOS EEPROM software: https://github.com/costarc/msxcart_flash32k 2022-12-25"
- moved on the sheet: R5, R7

Commit message: Updated footprint to r1 (smaller size & 3 holes)- better fit for Patola case
Parts:
- removed J2: WRITE_EN, Connector_PinHeader_2.54mm:PinHeader_1x02_P2.54mm_Vertical, symbol Connector_Generic:Conn_02x01
- JP1: footprint Roni Footprints:MSX_CART_SW -> Roni Footprints:MSX_CART_SW_Official_3Holes
Connections:
- net /MEM_WE is gone; now on net /WR: R5.1, U1.27 (~{WE})
Other:
- note added: "MSXPi Interface V1.0.1 Rev.3 RCC @ 2017 - 2023 MSXPi interface - connect MSX computer to Raspberry Pi EEPROM AT28C256 re-writeatable from MSX-DOS EEPROM software: https://github.com/costarc/msxcart_flash32k 2023-03-17"
- note removed: "MSXPi Interface V1.0.1 Rev.2 RCC @ 2017 - 2023 MSXPi interface - connect MSX computer to Raspberry Pi EEPROM AT28C256 re-writeatable from MSX-DOS EEPROM software: https://github.com/costarc/msxcart_flash32k 2023-02-26"
Changed lines of the file:
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@@
     (effects (font (size 1 1)) (justify left bottom))
   )
-  (text "MSXPi Interface V1.0.1 Rev.2\nRCC @ 2017 - 2023\n\nMSXPi interface - connect MSX computer to Raspberry Pi\nEEPROM AT28C256 re-writeatable from MSX-DOS\nEEPROM software: https://github.com/costarc/msxcart_flash32k\n\n2023-02-26"
+  (text "MSXPi Interface V1.0.1 Rev.3\nRCC @ 2017 - 2023\n\nMSXPi interface - connect MSX computer to Raspberry Pi\nEEPROM AT28C256 re-writeatable from MSX-DOS\nEEPROM software: https://github.com/costarc/msxcart_flash32k\n\n2023-03-17"
     (at 210.058 197.612 0)
     (effects (font (size 1.27 1.27)) (justify left bottom))
@@
     )
   )
-  (global_label "{slash}MEM_WE" (shape input) (at 161.29 154.94 270) (fields_autoplaced)
-    (effects (font (size 1.27 1.27)) (justify right))
-    (property "Intersheet References" "${INTERSHEET_REFS}" (id 0) (at 161.2106 166.3036 90)
+  (global_label "{slash}WR" (shape input) (at 161.29 154.94 270) (fields_autoplaced)
+    (effects (font (size 1.27 1.27)) (justify right))
+    (property "Intersheet References" "${INTERSHEET_REFS}" (id 0) (at 161.2106 161.405 90)
       (effects (font (size 1.27 1.27)) (justify right) hide)
     )
@@
     )
   )
-  (global_label "{slash}MEM_WE" (shape input) (at 167.64 125.73 0) (fields_autoplaced)
-    (effects (font (size 1.27 1.27)) (justify left))
-    (property "Intersheet References" "${INTERSHEET_REFS}" (id 0) (at 179.0036 125.6506 0)
-      (effects (font (size 1.27 1.27)) (justify left) hide)
-    )
-  )
   (global_label "SPI_RDY" (shape input) (at 196.342 120.396 180) (fields_autoplaced)
     (effects (font (size 1.27 1.27)) (justify right))
@@
     )
   )
-  (global_label "{slash}MEM_WE" (shape input) (at 149.86 66.802 180) (fields_autoplaced)
-    (effects (font (size 1.27 1.27)) (justify right))
-    (property "Intersheet References" "${INTERSHEET_REFS}" (id 0) (at 138.4964 66.7226 0)
+  (global_label "{slash}WR" (shape input) (at 149.86 66.802 180) (fields_autoplaced)
+    (effects (font (size 1.27 1.27)) (justify right))
+    (property "Intersheet References" "${INTERSHEET_REFS}" (id 0) (at 143.395 66.7226 0)
       (effects (font (size 1.27 1.27)) (justify right) hide)
     )
@@
     (effects (font (size 1.27 1.27)) (justify right))
     (property "Intersheet References" "${INTERSHEET_REFS}" (id 0) (at 68.5739 79.4226 0)
-      (effects (font (size 1.27 1.27)) (justify right) hide)
-    )
-  )
-  (global_label "{slash}WR" (shape input) (at 154.94 125.73 180) (fields_autoplaced)
-    (effects (font (size 1.27 1.27)) (justify right))
-    (property "Intersheet References" "${INTERSHEET_REFS}" (id 0) (at 148.475 125.6506 0)
       (effects (font (size 1.27 1.27)) (justify right) hide)
     )
@@
     (pin "1")
   )
-  (symbol (lib_id "Connector_Generic:Conn_02x01") (at 160.02 125.73 0) (unit 1)
-    (in_bom yes) (on_board yes)
-    (property "Reference" "J2" (id 0) (at 161.29 129.54 0))
-    (property "Value" "WRITE_EN" (id 1) (at 161.29 114.046 0)
-      (effects (font (size 1.27 1.27)) hide)
-    )
-    (property "Footprint" "Connector_PinHeader_2.54mm:PinHeader_1x02_P2.54mm_Vertical" (id 2) (at 160.02 125.73 0)
-      (effects (font (size 1.27 1.27)) hide)
-    )
-    (property "Datasheet" "~" (id 3) (at 160.02 125.73 0)
-      (effects (font (size 1.27 1.27)) hide)
-    )
-    (pin "1")
-    (pin "2")
-  )
   (symbol (lib_id "msxpi-eagle-import:CPOL-EUE2.5-5") (at 124.968 155.702 180) (unit 1)
     (in_bom yes) (on_board yes)
@@
       (effects (font (size 1.27 1.27)) hide)
     )
-    (property "Footprint" "Roni Footprints:MSX_CART_SW" (id 2) (at 92.456 56.642 0)
+    (property "Footprint" "Roni Footprints:MSX_CART_SW_Official_3Holes" (id 2) (at 92.456 56.642 0)
       (effects (font (size 1.27 1.27)) hide)
     )
@@
       (reference "J1") (unit 1) (value "ROM_SWITCH") (footprint "Connector_PinHeader_2.54mm:PinHeader_2x03_P2.54mm_Vertical")
     )
-    (path "/8ff8fd2b-89ae-4882-8211-de345c0da1ec"
-      (reference "J2") (unit 1) (value "WRITE_EN") (footprint "Connector_PinHeader_2.54mm:PinHeader_1x02_P2.54mm_Vertical")
-    )
     (path "/dc6b1a8c-9a10-4556-b1d7-411bee3b766e"
-      (reference "JP1") (unit 1) (value "MSXCART1") (footprint "Roni Footprints:MSX_CART_SW")
+      (reference "JP1") (unit 1) (value "MSXCART1") (footprint "Roni Footprints:MSX_CART_SW_Official_3Holes")
     )
     (path "/610fb86f-39b8-496e-b00e-193fd857bffc"
