File: hardware/Schematic/MSXPi_v1.1/msxpi.kicad_sch (KiCad schematic)
At the start: 35 parts, among them IC1 LD117A, J1 ROM_SWITCH, U1 AT28C256

Commit message: Updated Interface schema / pcb to v1.1Rev.0
Parts:
- removed +5V1, GND5, MOUNTHOLE1, MOUNTHOLE2, MOUNTHOLE3, MOUNTHOLE4, MOUNTHOLE5: 2,15/1,0, msxpi:2,15_1,0, symbol msxpi-eagle-import:2,15/1,0
- removed C6: 0.1uf, msxpi:C2.5-3, symbol msxpi-eagle-import:C2,5-3
- removed C9: 100uf, msxpi:E2,5-5, symbol msxpi-eagle-import:CPOL-EUE2.5-5
- removed SPI_CLK_PI_GPIO1: SPI_CLK, msxpi:2,15_1,0, symbol msxpi-eagle-import:2,15/1,0
- removed SPI_CS_PI_GPIO1: SPI_CS, msxpi:2,15_1,0, symbol msxpi-eagle-import:2,15/1,0
- removed SPI_MISO_PI_GPIO1: SPI_MISO, msxpi:2,15_1,0, symbol msxpi-eagle-import:2,15/1,0
- removed SPI_MOSI_PI_GPIO1: SPI_MOSI, msxpi:2,15_1,0, symbol msxpi-eagle-import:2,15/1,0
- removed SPI_RDY_PI_GPIO1: SPI_RDY, msxpi:2,15_1,0, symbol msxpi-eagle-import:2,15/1,0
- added C7: 0.1uf, msxpi:C2.5-3, symbol msxpi-eagle-import:C2,5-3
- added J4: Raspberry Pi GPIO, Roni Footprints:PinSocket_2x20_P2.54mm_Vertical, symbol Connector_Generic_MountingPin:Conn_02x20_Odd_Even_MountingPin
- added JP3, JP4, JP5, JP6: Jumper_3_Open, Jumper:SolderJumper-3_P1.3mm_Open_Pad1.0x1.5mm, symbol Jumper:Jumper_3_Open
- C1: value 100nf -> 0.1uf
- C2: renamed from C3; value 100nf -> 0.1uf
- C8: renamed from C2; value 100uf -> 0.1uf
- renumbered C4 to C3, C5 to C4, C7 to C5, C8 to C6, JP1 to J1, JP2 to J2, J1 to J3, R7 to R6, R8 to R7, IC1 to U1, EPM3064ALC44 to U2, U1 to U3
Connections:
- net +5V: now also C7.2, J4.2 (Pin_2), J4.4 (Pin_4)
- net GNDREF: now also C7.1, J4.6 (Pin_6)
- net SPI_CLK: now also JP4.2 (C)
- net SPI_CS: now also JP3.2 (C)
- net SPI_MISO: now also JP6.2 (C)
- net SPI_MOSI: now also JP5.2 (C)
- net SPI_RDY: now also J4.22 (Pin_22)
- new net nSPI_CLK: J4.23 (Pin_23), JP4.3 (B)
- new net nSPI_CS: J4.24 (Pin_24), JP3.3 (B)
- new net nSPI_MISO: J4.21 (Pin_21), JP6.3 (B)
- new net nSPI_MOSI: J4.19 (Pin_19), JP5.3 (B)
- new net oSPI_CLK: J4.38 (Pin_38), JP4.1 (A)
- new net oSPI_CS: J4.40 (Pin_40), JP3.1 (A)
- new net oSPI_MISO: J4.32 (Pin_32), JP6.1 (A)
- new net oSPI_MOSI: J4.36 (Pin_36), JP5.1 (A)
- no-connect marks 15 -> 10
Other:
- note added: "MSXPi Interface V1.1 Rev.0 RCC @ 2017 - 2023 MSXPi interface - connect MSX computer to Raspberry Pi EEPROM AT28C256 re-writeatable from MSX-DOS EEPROM software: https://github.com/costarc/msxcart_flash32k 2023-04-15"
- note removed: "MSXPi Interface V1.0.1 Rev.3 RCC @ 2017 - 2023 MSXPi interface - connect MSX computer to Raspberry Pi EEPROM AT28C256 re-writeatable from MSX-DOS EEPROM software: https://github.com/costarc/msxcart_flash32k 2023-03-17"
- note removed: "Mounting holes for RPI"
- note removed: "Solder pads for the Raspberry Pi"
- moved on the sheet: C1, C2, C3, C4, C5, C6, C8, J1, J2, J3, LED1, R1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
